Commit message: fix error in robot model related to wheel positions

File: src/robot_sbem/description/robot_sbem.urdf.xacro (robot description, xacro)
@@ -102,5 +102,5 @@
     <parent link="base_link"/>
     <child link="left_wheel"/>
-    <origin xyz="-0.075 0.175 0" rpy="-${pi/2} 0 0" />
+    <origin xyz="-0.075 -0.175 0" rpy="${pi/2} 0 0" />
     <axis xyz="0 0 5"/>
 </joint>
@@ -128,5 +128,5 @@
     <parent link="base_link"/>
     <child link="right_wheel"/>
-    <origin xyz="-0.075 -0.175 0" rpy="${pi/2} 0 0" />
+    <origin xyz="-0.075 0.175 0" rpy="${pi/2} 0 0" />
     <axis xyz="0 0 -1"/>
 </joint>

File: src/robot_sbem/description/ros2_control.xacro (robot description, xacro)
@@ -33,4 +33,5 @@
             <sensor name="battery_state">
                 <state_interface name="voltage" />
+                <state_interface name="current" />
             </sensor>
         </ros2_control>

Commit message: latest changes

File: src/robot_sbem/description/robot_sbem.urdf.xacro (robot description, xacro)
@@ -102,5 +102,5 @@
     <parent link="base_link"/>
     <child link="left_wheel"/>
-    <origin xyz="-0.075 -0.175 0" rpy="${pi/2} 0 0" />
+    <origin xyz="-0.075 0.175 0" rpy="-${pi/2} 0 0" />
     <axis xyz="0 0 5"/>
 </joint>
@@ -128,5 +128,5 @@
     <parent link="base_link"/>
     <child link="right_wheel"/>
-    <origin xyz="-0.075 0.175 0" rpy="${pi/2} 0 0" />
+    <origin xyz="-0.075 -0.175 0" rpy="${pi/2} 0 0" />
     <axis xyz="0 0 -1"/>
 </joint>
