Commit message: fix wrong orientation

File: src/robot_sbem/description/robot_core.xacro (robot description, xacro)
@@ -77,6 +77,6 @@
     <parent link="base_link"/>
     <child link="left_wheel"/>
-    <origin xyz="-0.075 0.175 0" rpy="-${pi/2} 0 0" />
-    <axis xyz="0 0 5"/>
+    <origin xyz="-0.075 0.175 0" rpy="0 ${pi/2} 0" />
+    <axis xyz="0 1 0"/>
 </joint>
 <link name="left_wheel">
@@ -103,6 +103,6 @@
     <parent link="base_link"/>
     <child link="right_wheel"/>
-    <origin xyz="-0.075 -0.175 0" rpy="${pi/2} 0 0" />
-    <axis xyz="0 0 -1"/>
+    <origin xyz="-0.075 -0.175 0" rpy="0 ${pi/2} 0" />
+    <axis xyz="0 1 0"/>
 </joint>
 <link name="right_wheel">
