Commit message: camera urdf changes

File: src/robot_sbem/description/camera.xacro (robot description, xacro)
@@ -3,8 +3,8 @@
     <joint name="camera_joint" type = "fixed">
         <parent link="chassis"/>
-        <child link="camera_link"/>
-        <origin xyz="0.23 0.0 0.065" rpy="0.0 0 0"/> <!-- 0.0 0 -${pi}-->
+        <child link="camera0_link"/>
+        <origin xyz="0.23 0.0 0.225" rpy="0.0 0 0"/> <!-- 0.0 0 -${pi}-->
     </joint>
-    <link name="camera_link">
+    <link name="camera0_link">
         <visual>
             <geometry>
@@ -18,5 +18,5 @@
     </link>
     <joint name="camera_optical_joint" type = "fixed">
-        <parent link="camera_link"/>
+        <parent link="camera0_link"/>
         <child link="camera_link_optical"/>
         <origin xyz="0 0.0 0" rpy="${-pi/2} 0 ${-pi/2}"/> <!-- 0.0 0 -${pi}-->
@@ -24,5 +24,5 @@
     <link name="camera_link_optical">
     </link>
-    <gazebo reference="camera_link">
+    <gazebo reference="camera0_link">
         <material>Gazebo/Red</material>
         <sensor name="camera" type="camera">
