Commit message: fix lidar orientation

File: src/sbem_description/description/robot_core.xacro (robot description, xacro)
@@ -22,4 +22,12 @@
   </collision>
 </link>
+<!-- BASE FOOTPRINT LINK -->
+<joint name="base_footprint_joint" type="fixed">
+    <parent link="base_link"/>
+    <child link="base_footprint"/>
+    <origin xyz="0 0 0" rpy="0 0 0"/>
+</joint>
+<link name="base_footprint">
+</link>
 <link name="cover_frame_1">
   <inertial>
@@ -284,5 +292,5 @@
   <child link="camera_1"/>
 </joint>
-<joint name="joint_castor_wheel_front" type="continuous">
+<joint name="joint_castor_wheel_front" type="fixed">
   <origin xyz="0.148231 0.0 -0.036123" rpy="0 0 0"/>
   <parent link="base_link"/>
@@ -290,5 +298,5 @@
   <axis xyz="0.0 -0.0 -1.0"/>
 </joint>
-<joint name="joint_castor_wheel_front_2" type="continuous">
+<joint name="joint_castor_wheel_front_2" type="fixed">
   <origin xyz="-0.018973 -0.009866 -0.029977" rpy="0 0 0"/>
   <parent link="support_castor_front_2"/>
@@ -296,5 +304,5 @@
   <axis xyz="-0.0 1.0 -0.0"/>
 </joint>
-<joint name="joint_castor_wheel_back" type="continuous">
+<joint name="joint_castor_wheel_back" type="fixed">
   <origin xyz="-0.154231 7.6e-05 -0.036123" rpy="0 0 0"/>
   <parent link="base_link"/>
@@ -302,5 +310,5 @@
   <axis xyz="0.0 -0.0 -1.0"/>
 </joint>
-<joint name="joint_castor_wheel_back_2" type="continuous">
+<joint name="joint_castor_wheel_back_2" type="fixed">
   <origin xyz="-0.018973 -0.009866 -0.029977" rpy="0 0 0"/>
   <parent link="support_castor_back_1"/>
@@ -309,5 +317,5 @@
 </joint>
 <joint name="laser_joint" type="fixed">
-  <origin xyz="0.176869 0.018946 0.0182" rpy="0 0 0"/>
+  <origin xyz="0.176869 0.018946 0.0182" rpy="0 0 -${pi}"/>
   <parent link="cover_frame_1"/>
   <child link="laser_frame"/>
